File: Ćevapad/Ćevapad.kicad_pcb (KiCad board)
At the start: 2 copper layers, 38 parts, among them SW1 RotaryEncoder_Switch, SW2 RotaryEncoder_Switch, SW3 RotaryEncoder_Switch, U1 SuperMini nRF52840, U2 TXS0101DBV

Commit message: Kicad Schematics & Roughing Board Layout
Parts:
- moved U1 10.2 mm to (84.0, 61.8)
Other:
- board outline added: 148 x 76.2 mm

Commit message: sdf
Parts:
- removed D17: SK6812, LED_SMD:LED_SK6812_PLCC4_5.0x5.0mm_P3.2mm
- removed U2: TXS0101DBV, Package_TO_SOT_SMD:SOT-23-6
- added H1: MountingHole, MountingHole:MountingHole_2.2mm_M2_ISO7380_Pad, F.Cu at (131.0, 82.2)
- added H2: MountingHole, MountingHole:MountingHole_2.2mm_M2_ISO7380_Pad, F.Cu at (174.8, 82.2)
- added H3: MountingHole, MountingHole:MountingHole_2.2mm_M2_ISO7380_Pad, F.Cu at (87.1, 107.5)
- added H4: MountingHole, MountingHole:MountingHole_2.2mm_M2_ISO7380_Pad, F.Cu at (87.1, 56.8)
- added H5: MountingHole, MountingHole:MountingHole_2.2mm_M2_ISO7380_Pad, F.Cu at (174.8, 107.5)
- added J1: OLED_128x64, ScottoKeebs_Components:OLED_128x64, F.Cu at (188.1, 46.1)
- moved U1 12.9 mm to (73.8, 53.8)
- turned SW1 to 180 degrees
- turned SW2 to 180 degrees
Other:
- board size 148 x 76.2 mm -> 145 x 76.2 mm
