File: Ćevapad/Ćevapad.kicad_sch (KiCad schematic)
At the start: 38 parts, among them SW1 RotaryEncoder_Switch, SW2 RotaryEncoder_Switch, SW3 RotaryEncoder_Switch, U1 SuperMini nRF52840, U2 TXS0101DBV

Commit message: sdf
Parts:
- removed D17: SK6812, LED_SMD:LED_SK6812_PLCC4_5.0x5.0mm_P3.2mm, symbol LED:SK6812
- added D17: SK6812MINI, LED_SMD:LED_SK6812MINI_PLCC4_3.5x3.5mm_P1.75mm, symbol LED:SK6812MINI
- added H1, H2, H3, H4, H5: MountingHole, MountingHole:MountingHole_2.2mm_M2_ISO7380_Pad, symbol Mechanical:MountingHole
- added J1: OLED_128x64, ScottoKeebs_Components:OLED_128x64, symbol ScottoKeebs:OLED_128x64
Other:
- moved on the sheet: SW1, SW2, SW3
